File: OMiGaS_Rev_3.kicad_sch (KiCad schematic)
At the start: 122 parts, among them J1 SMB, J2 Conn_2x5_P, J3 Conn_2x5_S, P1 Eink-display, Q1 NMOS_GSD, Q2 NMOS_GSD, SW1 SW_Push, U1 TMP117, U10 TPS22919DCKR, U11 MAX31329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

Commit message: Added BOM, optimized trim pot position, re-generated gerber
Parts:
- BT2: Manufacturer_Part_Number (none) -> BAT-HLD-012-SMT
- C1, C2, C3, C4: Comments (none) -> COG dialectic; Manufacturer_Part_Number (none) -> C1608C0G2A103J080AC
- C37, C39: Manufacturer_Part_Number (none) -> TPSA475M010R1400
- C8: Comments (none) -> Preferably film caps; Manufacturer_Part_Number (none) -> ECH-U1C102GX5
- D1, D2, D3, D6: Manufacturer_Part_Number (none) -> PMEG2005EJ-QX
- D4: Manufacturer_Part_Number (none) -> PMEG3010ER,115
- D5: Manufacturer_Part_Number (none) -> V2PL45HM3/H
- L1: Manufacturer_Part_Number (none) -> NRS5024T2R2NMGJ
- L2: Manufacturer_Part_Number (none) -> VLCF5020T-470MR40
- LED1: Manufacturer_Part_Number (none) -> 150060AS75000
- Q1, Q2: Manufacturer_Part_Number (none) -> T2N7002AK,LM
- RV1: Manufacturer_Part_Number (none) -> TC33X-2-104G
- RV3: Manufacturer_Part_Number (none) -> 3214W-1-104E
- SiPM1: Manufacturer_Part_Number (none) -> MICROFC-60035-SMT-TR
- U1: Manufacturer_Part_Number (none) -> TMP117MAIDRVR
- U10: Manufacturer_Part_Number TPS22919DCKR -> TPS22919DCKR
- U11: Manufacturer_Part_Number (none) -> MAX31329ELB+
- U12, U13: Manufacturer_Part_Number (none) -> LM7705MMX/NOPB
- U14: Manufacturer_Part_Number (none) -> SN74LVC3G17DCTRE4
- U15: Manufacturer_Part_Number (none) -> ADS1015IDGSR
- U2: Manufacturer_Part_Number M24C16-FMC6TG -> M24C04-RMC6TG
- U3, U4: Manufacturer_Part_Number (none) -> OPA2356AIDR
- U5: Manufacturer_Part_Number (none) -> 74LVC1G17GW,125
- U6: Manufacturer_Part_Number MAX16150BUT+T -> MAX16150AUT+T
- U8: Manufacturer_Part_Number TPS7A2045PDBVR -> TPS7A2045PDBVR
- U9: Manufacturer_Part_Number LT3462ES6#TRMPBF -> LT3462ES6#TRMPBF

Commit message: Updated BOM, added 3d model for B2B connector, corrected detector shell position
Parts:
- J2: Comments (none) -> Molex 524651070 compatible
- J3: Comments (none) -> Warning: This socket is NOT compatible with Molex 533091070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
Changed lines of the file:
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@@
 			)
 		)
-		(property "Comments" ""
+		(property "Comments" "Warning: This socket is NOT compatible with Molex 533091070, the snap height (actually weidth) is different"
 			(at 38.1 39.37 0)
 			(effects
@@
 			)
 		)
-		(property "Comments" ""
+		(property "Comments" "Molex 524651070 compatible"
 			(at 38.1 111.76 0)
 			(effects

Commit message: updated BOM
Parts:
- C1, C2, C3, C4: Comments COG dialectic -> C0G dialectic
Changed lines of the file:
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@@
 			)
 		)
-		(property "Comments" "COG dialectic"
+		(property "Comments" "C0G dialectic"
 			(at 88.9 38.1 0)
 			(effects
@@
 			)
 		)
-		(property "Comments" "COG dialectic"
+		(property "Comments" "C0G dialectic"
 			(at 78.74 38.1 0)
 			(effects
@@
 			)
 		)
-		(property "Comments" "COG dialectic"
+		(property "Comments" "C0G dialectic"
 			(at 99.06 38.1 0)
 			(effects
@@
 			)
 		)
-		(property "Comments" "COG dialectic"
+		(property "Comments" "C0G dialectic"
 			(at 109.22 38.1 0)
 			(effects

Commit message: fixed typo in BOM
Parts:
- C1, C2, C3, C4: Comments C0G dialectic -> C0G dielectic
Changed lines of the file:
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@@
 			)
 		)
-		(property "Comments" "C0G dialectic"
+		(property "Comments" "C0G dielectic"
 			(at 88.9 38.1 0)
 			(effects
@@
 			)
 		)
-		(property "Comments" "C0G dialectic"
+		(property "Comments" "C0G dielectic"
 			(at 78.74 38.1 0)
 			(effects
@@
 			)
 		)
-		(property "Comments" "C0G dialectic"
+		(property "Comments" "C0G dielectic"
 			(at 99.06 38.1 0)
 			(effects
@@
 			)
 		)
-		(property "Comments" "C0G dialectic"
+		(property "Comments" "C0G dielectic"
 			(at 109.22 38.1 0)
 			(effects
