File: OMiGaS_Rev_3.kicad_pcb (KiCad board)
At the start: 4 copper layers, 92 x 44 mm, 134 parts, among them J1 SMB, J2 Conn_2x5_P, J3 Conn_2x5_S, P1 Eink-display, Q1 NMOS_GSD, Q2 NMOS_GSD, SW1 SW_Push, U1 TMP117, U10 TPS22919DCKR, U11 MAX31329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

Commit message: Added BOM, optimized trim pot position, re-generated gerber
Parts:
- moved RV3 0.30 mm to (118.0, 139.3)
Routing:
- net Net-(R16-Pad1): track 4.91 -> 5.44 mm
Other:
- board text added: "3.3.2"
- board text removed: "3.3.1"

Commit message: changed to through hole pogo pin, improved ground stitching
Routing:
- net GND: vias 51 -> 71
Other:
- board text added: "3.3.3"
- board text removed: "3.3.2"
